Commit message: simulation ok

File: diffbot_description/urdf/diffbot.urdf_copy.xacro (robot description, xacro)
@@ -7,10 +7,6 @@
   <xacro:include filename="$(find ${package_name})/urdf/include/common_sensors.xacro" />
   <xacro:include filename="$(find ${package_name})/urdf/include/robot.gazebo.xacro" />
-  <!-- <xacro:property name="caster_wheel_yaml" value="$(find ${package_name})/config/${robot_name}/caster_wheel.yaml" />
-  <xacro:property name="caster_wheel_props" value="${xacro.load_yaml(caster_wheel_yaml)}"/> -->
   <xacro:property name="front_wheel_yaml" value="$(find ${package_name})/config/${robot_name}/front_wheel.yaml" />
   <xacro:property name="front_wheel_props" value="${xacro.load_yaml(front_wheel_yaml)}"/>
-  <!-- <xacro:property name="motor_yaml" value="$(find ${package_name})/config/${robot_name}/motor.yaml" />
-  <xacro:property name="motor_props" value="${xacro.load_yaml(motor_yaml)}"/> -->
   <xacro:property name="base_yaml" value="$(find ${package_name})/config/${robot_name}/base.yaml" />
   <xacro:property name="base_props" value="${xacro.load_yaml(base_yaml)}"/>
@@ -23,8 +19,4 @@
     <origin xyz="0 0 0" rpy="0 0 0" />
   </xacro:base>
-  <!-- Back Caster Wheel -->
-  <!-- <xacro:caster_wheel prefix="rear" reflect="-1"
-                      wheel_props="${caster_wheel_props}">
-  </xacro:caster_wheel> -->
   <!-- Front Wheels -->
   <xacro:wheel prefix="front_right" reflect="-1"
@@ -36,13 +28,4 @@
                       base_props="${base_props}" >
   </xacro:wheel>
-  <!-- Motors -->
-  <!-- <xacro:motor prefix="right" reflect="-1"
-                      motor_props="${motor_props}"
-                      base_props="${base_props}" >
-  </xacro:motor>
-  <xacro:motor prefix="left" reflect="1"
-                      motor_props="${motor_props}"
-                      base_props="${base_props}" >
-  </xacro:motor> -->
   <!-- Sensors -->
   <xacro:laser prefix="rplidar" parent_link="base_link"

File: diffbot_description/urdf/include/common_macros.urdf.xacro (robot description, xacro)
@@ -189,7 +189,13 @@
     <collision>
       <origin xyz="0.0 0.0 0.0" rpy="0.0 0.0 0.0"/>
-      <geometry>
-        <box size="${base_prop['base']['x_size']} ${base_prop['base']['y_size']} ${base_prop['base']['z_size']}"/>
-      </geometry>
+        <geometry>
+          <!-- The folder path get a folder_name global parameter -->
+          <xacro:if value="${scale != '' }" >
+            <mesh filename="package://${package_name}/meshes/${robot_name}/${mesh}" scale="${scale}"/>
+          </xacro:if>
+          <xacro:if value="${scale == '' }" >
+            <mesh filename="package://${package_name}/meshes/${robot_name}/${mesh}" />
+          </xacro:if>
+        </geometry>
     </collision>
     </link>
